Commit message: Add files via upload

File: nx15a/urdf/nx15a.urdf (robot description, URDF)
Before this commit: robot nx15a, 18 links, 17 joints
Links:
- link Body: mass 0.346 -> 0.345
- link Leg_Mid_LF: mass 0.039138 -> 0.0389; geometry collision box size=0.032 0.014 0.0712; visual mesh filename=package://nx15a/stl/Leg_Mid_LH.stl
- link Leg_Mid_LR: mass 0.039138 -> 0.0389
- link Leg_Mid_RF: mass 0.039138 -> 0.0389
- link Leg_Mid_RR: mass 0.039138 -> 0.0389
- link Leg_Upper_LF: mass 0.035143 -> 0.0343; geometry collision box size=0.018 0.0315 0.0422; visual mesh filename=package://nx15a/stl/Leg_Upper_LH.stl
- link Leg_Upper_LR: mass 0.035143 -> 0.0343; geometry collision box size=0.018 0.0315 0.0422; visual mesh filename=package://nx15a/stl/Leg_Upper_LH.stl
- link Leg_Upper_RF: mass 0.035143 -> 0.0343; geometry collision box size=0.018 0.0315 0.0422; visual mesh filename=package://nx15a/stl/Leg_Upper_RH.stl
- link Leg_Upper_RR: geometry collision box size=0.018 0.0315 0.0422; visual mesh filename=package://nx15a/stl/Leg_Upper_RH.stl
- link Leg_bottom_LF: mass 0.00816 -> 0.00773
- link Leg_bottom_LR: mass 0.00816 -> 0.00773
- link Leg_bottom_RF: mass 0.00816 -> 0.00773
- link Leg_bottom_RR: mass 0.00816 -> 0.00773
Joints:
- joint joint_LF_1: origin xyz=0.023 -0.0355 0 rpy=0 0 0 -> xyz=0.025 -0.0366 0 rpy=0 0 0
- joint joint_LF_2: origin xyz=0.013 0.021 -0.0093 rpy=0.785398163397 0 0 -> xyz=0.0119 0.022 -0.00965 rpy=0.785398163397 0 0
- joint joint_LF_3: origin xyz=0.022 0 -0.0707 rpy=-1.570796326795 0 0 -> xyz=0.023 0 -0.07085 rpy=-1.570796326795 0 0
- joint joint_LR_1: origin xyz=0.023 0.110 0 rpy=0 0 0 -> xyz=0.025 0.1089 0 rpy=0 0 0
- joint joint_LR_2: origin xyz=0.013 0.021 -0.0093 rpy=0.785398163397 0 0 -> xyz=0.0119 0.022 -0.00965 rpy=0.785398163397 0 0
- joint joint_LR_3: origin xyz=0.022 0 -0.0707 rpy=-1.570796326795 0 0 -> xyz=0.023 0 -0.07085 rpy=-1.570796326795 0 0
- joint joint_RF_1: origin xyz=-0.023 -0.0355 0 rpy=0 0 0 -> xyz=-0.025 -0.0366 0 rpy=0 0 0
- joint joint_RF_2: origin xyz=-0.013 0.021 -0.0093 rpy=0.785398163397 0 0 -> xyz=-0.0119 0.022 -0.00965 rpy=0.785398163397 0 0
- joint joint_RF_3: origin xyz=-0.022 0 -0.0707 rpy=-1.570796326795 0 0 -> xyz=-0.023 0 -0.07085 rpy=-1.570796326795 0 0
- joint joint_RR_1: origin xyz=-0.023 0.110 0 rpy=0 0 0 -> xyz=-0.025 0.1089 0 rpy=0 0 0
- joint joint_RR_2: origin xyz=-0.013 0.021 -0.0093 rpy=0.785398163397 0 0 -> xyz=-0.0119 0.022 -0.00965 rpy=0.785398163397 0 0
- joint joint_RR_3: origin xyz=-0.022 0 -0.0707 rpy=-1.570796326795 0 0 -> xyz=-0.023 0 -0.07085 rpy=-1.570796326795 0 0
